File: pcb/schematic/schematic.kicad_sch (KiCad schematic)
At the start: 31 parts, among them J1 284391-2, J2 284391-2, J3 284391-2, J4 284391-2, J5 USB_C_Receptacle_USB2.0_16P, K1 G5V-1, Q1 MMBT3904, SW1 BOOT_BTN, SW2 RESET_BTN, U1 ESP32-C3-WROOM-02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

Commit message: update footprint of C4 capacitor to 0805
Parts:
- C4: footprint (none) -> Capacitor_SMD:C_0805_2012Metric
Changed lines of the file:
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@@
 			)
 		)
-		(property "Footprint" ""
+		(property "Footprint" "Capacitor_SMD:C_0805_2012Metric"
 			(at 270.2052 45.72 0)
 			(effects
